File: Macropad9key.kicad_pcb (KiCad board)
At the start: 4 copper layers, 57.9 x 65.7 mm, 83 parts, among them J1 3220-10-0100-00, J2 4POS_2MM, J3 USB4085-GF-A, SW1 CherryMX_WithPCBPins, SW2 CherryMX_WithPCBPins, SW3 CherryMX_WithPCBPins, SW4 CherryMX_WithPCBPins, SW5 CherryMX_WithPCBPins, SW6 CherryMX_WithPCBPins, SW7 CherryMX_WithPCBPins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

Commit message: Add company and pcb name/rev to silk
Other:
- board text added: "LITTELL TECHNOLOGIES Macro9Pad REVA1"
